Commit message: Update myool_urdf - Original.urdf

File: urdf/myool_urdf - Original.urdf (robot description, URDF)
Before this commit: robot myool_urdf, 10 links, 9 joints
Links:
- removed link myool_battery
- removed link myool_front_left_wheel
- removed link myool_front_right_wheel
- removed link myool_rear_left_rocker
- removed link myool_rear_left_rocker_center_wheel
- removed link myool_rear_left_rocker_rear_wheel
- removed link myool_rear_right_rocker
- removed link myool_rear_right_rocker_center_wheel
- removed link myool_rear_right_rocker_rear_wheel
- link myool_chassis: geometry collision cylinder length=0.5 radius=1; visual mesh filename=package://myool_urdf/meshes/myool_chassis.STL
Joints:
- removed joint myool_battery_joint
- removed joint myool_front_left_joint
- removed joint myool_front_right_joint
- removed joint myool_rear_left_joint
- removed joint myool_rear_left_rocker_center_joint
- removed joint myool_rear_left_rocker_rear_joint
- removed joint myool_rear_right_joint
- removed joint myool_rear_right_rocker_center_joint
- removed joint myool_rear_right_rocker_rear_joint

Commit message: update

File: urdf/myool_urdf - Original.urdf (robot description, URDF)
Before this commit: robot myool_urdf, 1 links, 0 joints
Links:
- added link myool_battery, mass 0; collision mesh filename=package://myool_urdf/meshes/myool_battery.STL; visual mesh filename=package://myool_urdf/meshes/myool_battery.STL
- added link myool_front_left_wheel, mass 0.84556; collision mesh filename=package://myool_urdf/meshes/myool_front_left_wheel.STL; visual mesh filename=package://myool_urdf/meshes/myool_front_left_wheel.STL
- added link myool_front_right_wheel, mass 0.84556; collision mesh filename=package://myool_urdf/meshes/myool_front_right_wheel.STL; visual mesh filename=package://myool_urdf/meshes/myool_front_right_wheel.STL
- added link myool_rear_left_rocker, mass 0.32911; collision mesh filename=package://myool_urdf/meshes/myool_rear_left_rocker.STL; visual mesh filename=package://myool_urdf/meshes/myool_rear_left_rocker.STL
- added link myool_rear_left_rocker_center_wheel, mass 0.84556; collision mesh filename=package://myool_urdf/meshes/myool_rear_left_rocker_center_w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; visual mesh filename=package://myool_urdf/meshes/myool_rear_left_rocker_center_w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
- added link myool_rear_left_rocker_rear_wheel, mass 0.84556; collision mesh filename=package://myool_urdf/meshes/myool_rear_left_rocker_rear_whe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; visual mesh filename=package://myool_urdf/meshes/myool_rear_left_rocker_rear_whe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
- added link myool_rear_right_rocker, mass 0.32911; collision mesh filename=package://myool_urdf/meshes/myool_rear_right_rocker.STL; visual mesh filename=package://myool_urdf/meshes/myool_rear_right_rocker.STL
- added link myool_rear_right_rocker_center_wheel, mass 0.84556; collision mesh filename=package://myool_urdf/meshes/myool_rear_right_rocker_center_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; visual mesh filename=package://myool_urdf/meshes/myool_rear_right_rocker_center_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
- added link myool_rear_right_rocker_rear_wheel, mass 0.84556; collision mesh filename=package://myool_urdf/meshes/myool_rear_right_rocker_rear_wh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; visual mesh filename=package://myool_urdf/meshes/myool_rear_right_rocker_rear_wh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
- link myool_chassis: geometry collision mesh filename=package://myool_urdf/meshes/myool_chassis.STL; visual mesh filename=package://myool_urdf/meshes/myool_chassis.STL
Joints:
- added joint myool_battery_joint: type fixed, parent myool_chassis, child myool_battery, origin xyz=0.097493 0.025146 0.00635 rpy=0 0 0, axis 0 0 0
- added joint myool_front_left_joint: type continuous, parent myool_chassis, child myool_front_left_wheel, origin xyz=0.14829 0.21561 0.003175 rpy=0 0 0, axis 0 -1 0
- added joint myool_front_right_joint: type continuous, parent myool_chassis, child myool_front_right_wheel, origin xyz=0.14829 -0.21561 0.003175 rpy=0 0 0, axis 0 1 0
- added joint myool_rear_left_joint: type continuous, parent myool_chassis, child myool_rear_left_rocker, origin xyz=-0.15651 0.20097 0.003175 rpy=0 0 0, axis 0 1 0
- added joint myool_rear_left_rocker_center_joint: type continuous, parent myool_rear_left_rocker, child myool_rear_left_rocker_center_wheel, origin xyz=0.1016 0.01465 0 rpy=0 0 0, axis 0 -1 0
- added joint myool_rear_left_rocker_rear_joint: type continuous, parent myool_rear_left_rocker, child myool_rear_left_rocker_rear_wheel, origin xyz=-0.1016 0.01465 0 rpy=0 0 0, axis 0 -1 0
- added joint myool_rear_right_joint: type continuous, parent myool_chassis, child myool_rear_right_rocker, origin xyz=-0.15651 -0.20097 0.003175 rpy=0 0 0, axis 0 1 0
- added joint myool_rear_right_rocker_center_joint: type continuous, parent myool_rear_right_rocker, child myool_rear_right_rocker_center_wheel, origin xyz=0.1016 -0.01465 0 rpy=0 0 0, axis 0 1 0
- added joint myool_rear_right_rocker_rear_joint: type continuous, parent myool_rear_right_rocker, child myool_rear_right_rocker_rear_wheel, origin xyz=-0.1016 -0.01465 0 rpy=0 0 0, axis 0 1 0
