Commit message: chassis only urdf

File: urdf/myool_urdf.urdf (robot description, URDF)
Before this commit: robot myool_urdf, 10 links, 9 joints
Links:
- removed link myool_battery
- removed link myool_front_left_wheel
- removed link myool_front_right_wheel
- removed link myool_rear_left_rocker
- removed link myool_rear_left_rocker_center_wheel
- removed link myool_rear_left_rocker_rear_wheel
- removed link myool_rear_right_rocker
- removed link myool_rear_right_rocker_center_wheel
- removed link myool_rear_right_rocker_rear_wheel
Joints:
- removed joint myool_battery_joint
- removed joint myool_front_left_joint
- removed joint myool_front_right_joint
- removed joint myool_rear_left_joint
- removed joint myool_rear_left_rocker_center_joint
- removed joint myool_rear_left_rocker_rear_joint
- removed joint myool_rear_right_joint
- removed joint myool_rear_right_rocker_center_joint
- removed joint myool_rear_right_rocker_rear_joint

Commit message: Update myool_urdf.urdf

File: urdf/myool_urdf.urdf (robot description, URDF)
Before this commit: robot myool_urdf, 1 links, 0 joints
Links:
- link myool_chassis: mass 2.8701 -> None

Commit message: Update myool_urdf.urdf

File: urdf/myool_urdf.urdf (robot description, URDF)
Before this commit: robot myool_urdf, 1 links, 0 joints
Links:
- link myool_chassis: mass None -> 2.8701

Commit message: Update myool_urdf.urdf

File: urdf/myool_urdf.urdf (robot description, URDF)
Before this commit: robot myool_urdf, 1 links, 0 joints
Links:
- removed link myool_chassis
- added link myool_battery, mass 0; collision mesh filename=package://myool_urdf/meshes/myool_battery.STL; visual mesh filename=package://myool_urdf/meshes/myool_battery.STL
Joints:
- added joint myool_battery_joint: type fixed, parent myool_chassis, child myool_battery, origin xyz=0.097493 0.025146 0.00635 rpy=0 0 0, axis 0 0 0

Commit message: Update myool_urdf.urdf

File: urdf/myool_urdf.urdf (robot description, URDF)
Before this commit: robot myool_urdf, 1 links, 1 joints
Joints:
- removed joint myool_battery_joint

Commit message: Update myool_urdf.urdf

File: urdf/myool_urdf.urdf (robot description, URDF)
Before this commit: robot myool_urdf, 1 links, 0 joints
Links:
- added link myool_chassis, mass 2.8701; collision mesh filename=package://myool_urdf/meshes/myool_chassis.STL; visual mesh filename=package://myool_urdf/meshes/myool_chassis.STL
- added link myool_front_left_wheel, mass 0.84556; collision mesh filename=package://myool_urdf/meshes/myool_front_left_wheel.STL; visual mesh filename=package://myool_urdf/meshes/myool_front_left_wheel.STL
- added link myool_front_right_wheel, mass 0.84556; collision mesh filename=package://myool_urdf/meshes/myool_front_right_wheel.STL; visual mesh filename=package://myool_urdf/meshes/myool_front_right_wheel.STL
- added link myool_rear_left_rocker, mass 0.32911; collision mesh filename=package://myool_urdf/meshes/myool_rear_left_rocker.STL; visual mesh filename=package://myool_urdf/meshes/myool_rear_left_rocker.STL
- added link myool_rear_left_rocker_center_wheel, mass 0.84556; collision mesh filename=package://myool_urdf/meshes/myool_rear_left_rocker_center_w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; visual mesh filename=package://myool_urdf/meshes/myool_rear_left_rocker_center_w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
- added link myool_rear_left_rocker_rear_wheel, mass 0.84556; collision mesh filename=package://myool_urdf/meshes/myool_rear_left_rocker_rear_whe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; visual mesh filename=package://myool_urdf/meshes/myool_rear_left_rocker_rear_whe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
- added link myool_rear_right_rocker, mass 0.32911; collision mesh filename=package://myool_urdf/meshes/myool_rear_right_rocker.STL; visual mesh filename=package://myool_urdf/meshes/myool_rear_right_rocker.STL
- added link myool_rear_right_rocker_center_wheel, mass 0.84556; collision mesh filename=package://myool_urdf/meshes/myool_rear_right_rocker_center_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; visual mesh filename=package://myool_urdf/meshes/myool_rear_right_rocker_center_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
- added link myool_rear_right_rocker_rear_wheel, mass 0.84556; collision mesh filename=package://myool_urdf/meshes/myool_rear_right_rocker_rear_wh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; visual mesh filename=package://myool_urdf/meshes/myool_rear_right_rocker_rear_wh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
Joints:
- added joint myool_battery_joint: type fixed, parent myool_chassis, child myool_battery, origin xyz=0.097493 0.025146 0.00635 rpy=0 0 0, axis 0 0 0
- added joint myool_front_left_joint: type continuous, parent myool_chassis, child myool_front_left_wheel, origin xyz=0.14829 0.21561 0.003175 rpy=0 0 0, axis 0 -1 0
- added joint myool_front_right_joint: type continuous, parent myool_chassis, child myool_front_right_wheel, origin xyz=0.14829 -0.21561 0.003175 rpy=0 0 0, axis 0 1 0
- added joint myool_rear_left_joint: type continuous, parent myool_chassis, child myool_rear_left_rocker, origin xyz=-0.15651 0.20097 0.003175 rpy=0 0 0, axis 0 1 0
- added joint myool_rear_left_rocker_center_joint: type continuous, parent myool_rear_left_rocker, child myool_rear_left_rocker_center_wheel, origin xyz=0.1016 0.01465 0 rpy=0 0 0, axis 0 -1 0
- added joint myool_rear_left_rocker_rear_joint: type continuous, parent myool_rear_left_rocker, child myool_rear_left_rocker_rear_wheel, origin xyz=-0.1016 0.01465 0 rpy=0 0 0, axis 0 -1 0
- added joint myool_rear_right_joint: type continuous, parent myool_chassis, child myool_rear_right_rocker, origin xyz=-0.15651 -0.20097 0.003175 rpy=0 0 0, axis 0 1 0
- added joint myool_rear_right_rocker_center_joint: type continuous, parent myool_rear_right_rocker, child myool_rear_right_rocker_center_wheel, origin xyz=0.1016 -0.01465 0 rpy=0 0 0, axis 0 1 0
- added joint myool_rear_right_rocker_rear_joint: type continuous, parent myool_rear_right_rocker, child myool_rear_right_rocker_rear_wheel, origin xyz=-0.1016 -0.01465 0 rpy=0 0 0, axis 0 1 0

Commit message: Update myool_urdf.urdf

File: urdf/myool_urdf.urdf (robot description, URDF)
Before this commit: robot myool_urdf, 1 links, 0 joints
Links:
- link myool_chassis: geometry collision cylinder length=0.5 radius=1; visual cylinder length=0.5 radius=1

Commit message: Update myool_urdf.urdf

File: urdf/myool_urdf.urdf (robot description, URDF)
Before this commit: robot myool_urdf, 1 links, 0 joints
Links:
- link myool_chassis: geometry collision box size=0.42 0.41 0.08; visual box size=0.42 0.41 0.08

Commit message: Update myool_urdf.urdf

File: urdf/myool_urdf.urdf (robot description, URDF)
Before this commit: robot myool_urdf, 1 links, 0 joints
Links:
- link myool_chassis: geometry collision box size=0.42 0.345 0.08; visual box size=0.42 0.345 0.007

Commit message: Update myool_urdf.urdf

File: urdf/myool_urdf.urdf (robot description, URDF)
Before this commit: robot myool_urdf, 1 links, 0 joints
Links:
- added link myool_front_left_wheel, mass 0.84556; collision cylinder length=0.0435 radius=0.17; visual cylinder length=0.0435 radius=0.17
- added link myool_front_right_wheel, mass 0.84556; collision cylinder length=0.0435 radius=0.17; visual cylinder length=0.0435 radius=0.17
Joints:
- added joint myool_front_right_joint: type continuous, parent myool_chassis, child myool_front_right_wheel, origin xyz=0.14829 -0.21561 0.003175 rpy=0 0 0, axis 0 1 0

Commit message: Update myool_urdf.urdf

File: urdf/myool_urdf.urdf (robot description, URDF)
Before this commit: robot myool_urdf, 3 links, 1 joints
Links:
- removed link myool_front_left_wheel

Commit message: Update myool_urdf.urdf

File: urdf/myool_urdf.urdf (robot description, URDF)
Before this commit: robot myool_urdf, 2 links, 1 joints
Links:
- link myool_front_right_wheel: geometry collision cylinder length=0.0435 radius=0.85; visual cylinder length=0.0435 radius=0.17

Commit message: Update myool_urdf.urdf

File: urdf/myool_urdf.urdf (robot description, URDF)
Before this commit: robot myool_urdf, 2 links, 1 joints
Links:
- link myool_front_right_wheel: geometry collision cylinder length=0.0435 radius=0.085; visual cylinder length=0.0435 radius=0.17

Commit message: Update myool_urdf.urdf

File: urdf/myool_urdf.urdf (robot description, URDF)
Before this commit: robot myool_urdf, 2 links, 1 joints
Links:
- link myool_front_right_wheel: geometry collision cylinder length=0.0435 radius=0.085; visual cylinder length=0.0435 radius=0.085
Joints:
- joint myool_front_right_joint: origin xyz=0.14829 -0.21561 0.003175 rpy=0 0 0 -> xyz=0.14829 -0.21561 0.003175 rpy=90 0 0

Commit message: Update myool_urdf.urdf

File: urdf/myool_urdf.urdf (robot description, URDF)
Before this commit: robot myool_urdf, 2 links, 1 joints
Links:
- added link myool_front_left_wheel, mass 0.84556; collision cylinder length=0.0435 radius=0.085; visual cylinder length=0.0435 radius=0.085
Joints:
- added joint myool_front_left_joint: type continuous, parent myool_chassis, child myool_front_left_wheel, origin xyz=0.14829 0.21561 0.003175 rpy=90 0 0, axis 0 -1 0

Commit message: Update myool_urdf.urdf

File: urdf/myool_urdf.urdf (robot description, URDF)
Before this commit: robot myool_urdf, 3 links, 2 joints
Joints:
- joint myool_front_left_joint: origin xyz=0.14829 0.21561 0.003175 rpy=90 0 0 -> xyz=0.14829 0.21561 0.003175 rpy=0 0 0
- joint myool_front_right_joint: origin xyz=0.14829 -0.21561 0.003175 rpy=90 0 0 -> xyz=0.14829 -0.21561 0.003175 rpy=0 0 0

Commit message: Update myool_urdf.urdf

File: urdf/myool_urdf.urdf (robot description, URDF)
Before this commit: robot myool_urdf, 3 links, 2 joints
Links:
- added link myool_rear_right_rocker, mass 0.32911; collision box size=0.28 0.01 0.08; visual box size=0.28 0.01 0.08
- added link myool_rear_right_rocker_rear_wheel, mass 0.84556; collision cylinder length=0.0435 radius=0.085; visual cylinder length=0.0435 radius=0.085
Joints:
- added joint myool_rear_right_joint: type continuous, parent myool_chassis, child myool_rear_right_rocker, origin xyz=-0.15651 -0.20097 0.003175 rpy=0 0 0, axis 0 1 0
- added joint myool_rear_right_rocker_rear_joint: type continuous, parent myool_rear_right_rocker, child myool_rear_right_rocker_rear_wheel, origin xyz=-0.1016 -0.01465 0 rpy=0 0 0, axis 0 1 0

Commit message: Update myool_urdf.urdf

File: urdf/myool_urdf.urdf (robot description, URDF)
Before this commit: robot myool_urdf, 5 links, 4 joints
Links:
- added link myool_rear_left_rocker, mass 0.32911; collision box size=0.28 0.01 0.08; visual box size=0.28 0.01 0.08
- added link myool_rear_left_rocker_center_wheel, mass 0.84556; collision cylinder length=0.0435 radius=0.085; visual cylinder length=0.0435 radius=0.085
- added link myool_rear_left_rocker_rear_wheel, mass 0.84556; collision cylinder length=0.0435 radius=0.085; visual cylinder length=0.0435 radius=0.085
- added link myool_rear_right_rocker_center_wheel, mass 0.84556; collision cylinder length=0.0435 radius=0.085; visual cylinder length=0.0435 radius=0.085
Joints:
- added joint myool_rear_left_joint: type continuous, parent myool_chassis, child myool_rear_left_rocker, origin xyz=-0.15651 0.20097 0.003175 rpy=0 0 0, axis 0 1 0
- added joint myool_rear_left_rocker_center_joint: type continuous, parent myool_rear_left_rocker, child myool_rear_left_rocker_center_wheel, origin xyz=0.1016 0.01465 0 rpy=0 0 0, axis 0 -1 0
- added joint myool_rear_left_rocker_rear_joint: type continuous, parent myool_rear_left_rocker, child myool_rear_left_rocker_rear_wheel, origin xyz=-0.1016 0.01465 0 rpy=0 0 0, axis 0 -1 0
- added joint myool_rear_right_rocker_center_joint: type continuous, parent myool_rear_right_rocker, child myool_rear_right_rocker_center_wheel, origin xyz=0.1016 -0.01465 0 rpy=0 0 0, axis 0 1 0

Commit message: Update myool_urdf.urdf

File: urdf/myool_urdf.urdf (robot description, URDF)
Before this commit: robot myool_urdf, 9 links, 8 joints
Links:
- added link myool_battery, mass 0; collision box size=0.285 0.20 0.075; visual box size=0.285 0.20 0.075
Joints:
- added joint myool_battery_joint: type fixed, parent myool_chassis, child myool_battery, origin xyz=0.097493 0.025146 0.00635 rpy=0 0 0, axis 0 0 0

Commit message: Update myool_urdf.urdf

File: urdf/myool_urdf.urdf (robot description, URDF)
Before this commit: robot myool_urdf, 10 links, 9 joints
Joints:
- joint myool_battery_joint: origin xyz=0.097493 0.025146 0.00635 rpy=0 0 0 -> xyz=-0.097493 0.025146 0.00635 rpy=0 0 0

Commit message: Update myool_urdf.urdf

File: urdf/myool_urdf.urdf (robot description, URDF)
Before this commit: robot myool_urdf, 10 links, 9 joints
Joints:
- joint myool_battery_joint: origin xyz=-0.097493 0.025146 0.00635 rpy=0 0 0 -> xyz=0 0 0 rpy=0 0 0

Commit message: Update myool_urdf.urdf

File: urdf/myool_urdf.urdf (robot description, URDF)
Before this commit: robot myool_urdf, 10 links, 9 joints
Links:
- link myool_chassis: geometry collision box size=0.42 0.345 0.007; visual box size=0.42 0.345 0.007

Commit message: Update myool_urdf.urdf

File: urdf/myool_urdf.urdf (robot description, URDF)
Before this commit: robot myool_urdf, 10 links, 9 joints
Joints:
- joint myool_battery_joint: origin xyz=0 0 0 rpy=0 0 0 -> xyz=0 0 0.085 rpy=0 0 0

Commit message: Update myool_urdf.urdf

File: urdf/myool_urdf.urdf (robot description, URDF)
Before this commit: robot myool_urdf, 10 links, 9 joints
Joints:
- joint myool_battery_joint: origin xyz=0 0 0.085 rpy=0 0 0 -> xyz=0 0 0 rpy=0 0 0

Commit message: Update myool_urdf.urdf

File: urdf/myool_urdf.urdf (robot description, URDF)
Before this commit: robot myool_urdf, 10 links, 9 joints
Joints:
- joint myool_battery_joint: origin xyz=0 0 0 rpy=0 0 0 -> xyz=0 0 0.0375 rpy=0 0 0

Commit message: Update myool_urdf.urdf

File: urdf/myool_urdf.urdf (robot description, URDF)
Before this commit: robot myool_urdf, 10 links, 9 joints
Links:
- link myool_battery: mass 0 -> 7
- link myool_front_left_wheel: mass 0.84556 -> 3
- link myool_front_right_wheel: mass 0.84556 -> 3
- link myool_rear_left_rocker_center_wheel: mass 0.84556 -> 3
- link myool_rear_left_rocker_rear_wheel: mass 0.84556 -> 3
- link myool_rear_right_rocker_center_wheel: mass 0.84556 -> 3
- link myool_rear_right_rocker_rear_wheel: mass 0.84556 -> 3

Commit message: Update myool_urdf.urdf

File: urdf/myool_urdf.urdf (robot description, URDF)
Before this commit: robot myool_urdf, 10 links, 9 joints
Joints:
- joint myool_rear_left_rocker_center_joint: origin xyz=0.1016 0.01465 0 rpy=0 0 0 -> xyz=0.1016 0.0364 0 rpy=0 0 0
- joint myool_rear_left_rocker_rear_joint: origin xyz=-0.1016 0.01465 0 rpy=0 0 0 -> xyz=-0.1016 0.0364 0 rpy=0 0 0
- joint myool_rear_right_rocker_center_joint: origin xyz=0.1016 -0.01465 0 rpy=0 0 0 -> xyz=0.1016 -0.0364 0 rpy=0 0 0
- joint myool_rear_right_rocker_rear_joint: origin xyz=-0.1016 -0.01465 0 rpy=0 0 0 -> xyz=-0.1016 -0.0364 0 rpy=0 0 0

Commit message: Update myool_urdf.urdf

File: urdf/myool_urdf.urdf (robot description, URDF)
Before this commit: robot myool_urdf, 10 links, 9 joints
Joints:
- joint myool_front_left_joint: origin xyz=0.14829 0.21561 0.003175 rpy=0 0 0 -> xyz=0.14829 0.23736 0.003175 rpy=0 0 0
- joint myool_front_right_joint: origin xyz=0.14829 -0.21561 0.003175 rpy=0 0 0 -> xyz=0.14829 -0.23736 0.003175 rpy=0 0 0

Commit message: Update myool_urdf.urdf

File: urdf/myool_urdf.urdf (robot description, URDF)
Before this commit: robot myool_urdf, 10 links, 9 joints
Joints:
- joint myool_front_left_joint: axis 0 -1 0 -> 0 1 0; limit (none) -> effort=10000 velocity=1000
- joint myool_front_right_joint: limit (none) -> effort=10000 velocity=1000
- joint myool_rear_left_rocker_center_joint: axis 0 -1 0 -> 0 1 0; limit (none) -> effort=10000 velocity=1000
- joint myool_rear_left_rocker_rear_joint: axis 0 -1 0 -> 0 1 0; limit (none) -> effort=10000 velocity=1000
- joint myool_rear_right_rocker_center_joint: limit (none) -> effort=10000 velocity=1000
- joint myool_rear_right_rocker_rear_joint: limit (none) -> effort=10000 velocity=1000

Commit message: Update myool_urdf.urdf

File: urdf/myool_urdf.urdf (robot description, URDF)
Before this commit: robot myool_urdf, 10 links, 9 joints
Links:
- link myool_front_left_wheel: mass 3 -> 2.2
- link myool_front_right_wheel: mass 3 -> 2.2
- link myool_rear_left_rocker_center_wheel: mass 3 -> 2.2
- link myool_rear_left_rocker_rear_wheel: mass 3 -> 2.2
- link myool_rear_right_rocker_center_wheel: mass 3 -> 2.2
- link myool_rear_right_rocker_rear_wheel: mass 3 -> 2.2

Commit message: Update myool_urdf.urdf

File: urdf/myool_urdf.urdf (robot description, URDF)
Before this commit: robot myool_urdf, 10 links, 9 joints
Joints:
- joint myool_rear_right_joint: limit (none) -> upper=0.523; type continuous -> revolute

Commit message: Update myool_urdf.urdf

File: urdf/myool_urdf.urdf (robot description, URDF)
Before this commit: robot myool_urdf, 10 links, 9 joints
Joints:
- joint myool_rear_left_joint: limit (none) -> upper=0.523; type continuous -> revolute

Commit message: Update myool_urdf.urdf

File: urdf/myool_urdf.urdf (robot description, URDF)
Before this commit: robot myool_urdf, 10 links, 9 joints
Joints:
- joint myool_rear_left_joint: type revolute -> continuous
- joint myool_rear_right_joint: type revolute -> continuous

Commit message: Update myool_urdf.urdf

File: urdf/myool_urdf.urdf (robot description, URDF)
Before this commit: robot myool_urdf, 10 links, 9 joints
Joints:
- joint myool_rear_left_joint: limit effort=10000 velocity=1000 -> upper=0.523; type continuous -> revolute
- joint myool_rear_right_joint: type continuous -> revolute

Commit message: update

File: urdf/myool_urdf.urdf (robot description, URDF)
Before this commit: robot myool_urdf, 10 links, 9 joints
Joints:
- joint myool_rear_left_joint: limit upper=0.523 -> effort=10000 velocity=1000

Commit message: Update myool_urdf.urdf

File: urdf/myool_urdf.urdf (robot description, URDF)
Before this commit: robot myool_urdf, 10 links, 9 joints
Joints:
- joint myool_rear_left_joint: type continuous -> revolute

Commit message: Update myool_urdf.urdf

File: urdf/myool_urdf.urdf (robot description, URDF)
Before this commit: robot myool_urdf, 10 links, 9 joints
Joints:
- joint myool_rear_left_joint: limit effort=10000 velocity=1000 -> upper=0.523 effort=10000 velocity=1000

Commit message: Update myool_urdf.urdf

File: urdf/myool_urdf.urdf (robot description, URDF)
Before this commit: robot myool_urdf, 10 links, 9 joints
Joints:
- joint myool_rear_right_joint: origin xyz=-0.15651 -0.20097 0.003175 rpy=0 0 0 -> xyz=-0.15651 -0.20097 0.003175 rpy=0 0.392 0

Commit message: Update myool_urdf.urdf

File: urdf/myool_urdf.urdf (robot description, URDF)
Before this commit: robot myool_urdf, 10 links, 9 joints
Joints:
- joint myool_rear_right_joint: origin xyz=-0.15651 -0.20097 0.003175 rpy=0 0.392 0 -> xyz=-0.15651 -0.20097 0.003175 rpy=0 0 0

Commit message: Update myool_urdf.urdf

File: urdf/myool_urdf.urdf (robot description, URDF)
Before this commit: robot myool_urdf, 10 links, 9 joints
Joints:
- joint myool_front_left_joint: limit effort=10000 velocity=1000 -> effort=10000 velocity=10
- joint myool_front_right_joint: limit effort=10000 velocity=1000 -> effort=10000 velocity=10
- joint myool_rear_left_joint: limit upper=0.523 effort=10000 velocity=1000 -> upper=0.523 effort=10000 velocity=10
- joint myool_rear_left_rocker_center_joint: limit effort=10000 velocity=1000 -> effort=10000 velocity=10
- joint myool_rear_left_rocker_rear_joint: limit effort=10000 velocity=1000 -> effort=10000 velocity=10
- joint myool_rear_right_joint: limit upper=0.523 effort=10000 velocity=1000 -> upper=0.523 effort=10000 velocity=10
- joint myool_rear_right_rocker_center_joint: limit effort=10000 velocity=1000 -> effort=10000 velocity=10
- joint myool_rear_right_rocker_rear_joint: limit effort=10000 velocity=1000 -> effort=10000 velocity=10

Commit message: Update myool_urdf.urdf

File: urdf/myool_urdf.urdf (robot description, URDF)
Before this commit: robot myool_urdf, 10 links, 9 joints
Joints:
- joint myool_front_left_joint: limit effort=10000 velocity=10 -> effort=10000 velocity=100
- joint myool_front_right_joint: limit effort=10000 velocity=10 -> effort=10000 velocity=100
- joint myool_rear_left_joint: limit upper=0.523 effort=10000 velocity=10 -> upper=0.523 effort=10000 velocity=100
- joint myool_rear_left_rocker_center_joint: limit effort=10000 velocity=10 -> effort=10000 velocity=100
- joint myool_rear_left_rocker_rear_joint: limit effort=10000 velocity=10 -> effort=10000 velocity=100
- joint myool_rear_right_joint: limit upper=0.523 effort=10000 velocity=10 -> upper=0.523 effort=10000 velocity=100
- joint myool_rear_right_rocker_center_joint: limit effort=10000 velocity=10 -> effort=10000 velocity=100
- joint myool_rear_right_rocker_rear_joint: limit effort=10000 velocity=10 -> effort=10000 velocity=100

Commit message: Update myool_urdf.urdf

File: urdf/myool_urdf.urdf (robot description, URDF)
Before this commit: robot myool_urdf, 10 links, 9 joints
Joints:
- joint myool_front_left_joint: limit effort=10000 velocity=100 -> effort=10000 velocity=0
- joint myool_front_right_joint: limit effort=10000 velocity=100 -> effort=10000 velocity=0
- joint myool_rear_left_joint: limit upper=0.523 effort=10000 velocity=100 -> upper=0.523 effort=10000 velocity=0
- joint myool_rear_left_rocker_center_joint: limit effort=10000 velocity=100 -> effort=10000 velocity=0
- joint myool_rear_left_rocker_rear_joint: limit effort=10000 velocity=100 -> effort=10000 velocity=0
- joint myool_rear_right_joint: limit upper=0.523 effort=10000 velocity=100 -> upper=0.523 effort=10000 velocity=0
- joint myool_rear_right_rocker_center_joint: limit effort=10000 velocity=100 -> effort=10000 velocity=0
- joint myool_rear_right_rocker_rear_joint: limit effort=10000 velocity=100 -> effort=10000 velocity=0

Commit message: update

File: urdf/myool_urdf.urdf (robot description, URDF)
Before this commit: robot myool_urdf, 10 links, 9 joints
Joints:
- joint myool_front_left_joint: limit effort=10000 velocity=0 -> effort=10000 velocity=100
- joint myool_front_right_joint: limit effort=10000 velocity=0 -> effort=10000 velocity=100
- joint myool_rear_left_joint: limit upper=0.523 effort=10000 velocity=0 -> upper=0.523 effort=10000 velocity=100
- joint myool_rear_left_rocker_center_joint: limit effort=10000 velocity=0 -> effort=10000 velocity=100
- joint myool_rear_left_rocker_rear_joint: limit effort=10000 velocity=0 -> effort=10000 velocity=100
- joint myool_rear_right_joint: limit upper=0.523 effort=10000 velocity=0 -> upper=0.523 effort=10000 velocity=100
- joint myool_rear_right_rocker_center_joint: limit effort=10000 velocity=0 -> effort=10000 velocity=100
- joint myool_rear_right_rocker_rear_joint: limit effort=10000 velocity=0 -> effort=10000 velocity=100

Commit message: update

File: urdf/myool_urdf.urdf (robot description, URDF)
Before this commit: robot myool_urdf, 10 links, 9 joints
Links:
- removed link myool_chassis
- added link base_link, mass 2.8701; collision box size=0.42 0.345 0.007; visual box size=0.42 0.345 0.007
Joints:
- joint myool_battery_joint: parent myool_chassis -> base_link
- joint myool_front_left_joint: parent myool_chassis -> base_link
- joint myool_front_right_joint: parent myool_chassis -> base_link
- joint myool_rear_left_joint: parent myool_chassis -> base_link
- joint myool_rear_right_joint: parent myool_chassis -> base_link
